File: phase/phase.sch (KiCad schematic (older format))
At the start: 66 parts, among them J1 USB_C_Receptacle_USB2.0, J2 AudioJack4, K1 KEYSW, K10 KEYSW, K11 KEYSW, K12 KEYSW, K13 KEYSW, K14 KEYSW, K15 KEYSW, K16 KEYSW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

Commit message: renamed files to remove version number, add gitignore
Parts:
- D1, D10, D11, D12, D13, D14, D15, D16, D17, D18, D19, D2, D20, D21, D3, D4, D5, D6, D7, D8, D9: footprint phase_v1_0:D_SOD-123-dual -> phase:D_SOD-123-dual
- J2: footprint phase_v1_0:TRRS-PJ-320A-dual -> phase:TRRS-PJ-320A-dual
Changed lines of the file:
@@
 F 0 "D1" V 4746 1570 50  0000 R CNN
 F 1 "D" V 4655 1570 50  0000 R CNN
-F 2 "phase_v1_0:D_SOD-123-dual" H 4700 1650 50  0001 C CNN
+F 2 "phase:D_SOD-123-dual" H 4700 1650 50  0001 C CNN
 F 3 "~" H 4700 1650 50  0001 C CNN
 	1    4700 1650
@@
 F 0 "D2" V 4746 2070 50  0000 R CNN
 F 1 "D" V 4655 2070 50  0000 R CNN
-F 2 "phase_v1_0:D_SOD-123-dual" H 4700 2150 50  0001 C CNN
+F 2 "phase:D_SOD-123-dual" H 4700 2150 50  0001 C CNN
 F 3 "~" H 4700 2150 50  0001 C CNN
 	1    4700 2150
@@
 F 0 "D3" V 4746 2570 50  0000 R CNN
 F 1 "D" V 4655 2570 50  0000 R CNN
-F 2 "phase_v1_0:D_SOD-123-dual" H 4700 2650 50  0001 C CNN
+F 2 "phase:D_SOD-123-dual" H 4700 2650 50  0001 C CNN
 F 3 "~" H 4700 2650 50  0001 C CNN
 	1    4700 2650
@@
 F 0 "D18" V 9746 1570 50  0000 R CNN
 F 1 "D" V 9655 1570 50  0000 R CNN
-F 2 "phase_v1_0:D_SOD-123-dual" H 9700 1650 50  0001 C CNN
+F 2 "phase:D_SOD-123-dual" H 9700 1650 50  0001 C CNN
 F 3 "~" H 9700 1650 50  0001 C CNN
 	1    9700 1650
@@
 F 0 "D19" V 9746 2070 50  0000 R CNN
 F 1 "D" V 9655 2070 50  0000 R CNN
-F 2 "phase_v1_0:D_SOD-123-dual" H 9700 2150 50  0001 C CNN
+F 2 "phase:D_SOD-123-dual" H 9700 2150 50  0001 C CNN
 F 3 "~" H 9700 2150 50  0001 C CNN
 	1    9700 2150
@@
 F 0 "D20" V 9746 2570 50  0000 R CNN
 F 1 "D" V 9655 2570 50  0000 R CNN
-F 2 "phase_v1_0:D_SOD-123-dual" H 9700 2650 50  0001 C CNN
+F 2 "phase:D_SOD-123-dual" H 9700 2650 50  0001 C CNN
 F 3 "~" H 9700 2650 50  0001 C CNN
 	1    9700 2650
@@
 F 0 "D21" V 9746 3070 50  0000 R CNN
 F 1 "D" V 9655 3070 50  0000 R CNN
-F 2 "phase_v1_0:D_SOD-123-dual" H 9700 3150 50  0001 C CNN
+F 2 "phase:D_SOD-123-dual" H 9700 3150 50  0001 C CNN
 F 3 "~" H 9700 3150 50  0001 C CNN
 	1    9700 3150
@@
 F 0 "D17" V 8746 3070 50  0000 R CNN
 F 1 "D" V 8655 3070 50  0000 R CNN
-F 2 "phase_v1_0:D_SOD-123-dual" H 8700 3150 50  0001 C CNN
+F 2 "phase:D_SOD-123-dual" H 8700 3150 50  0001 C CNN
 F 3 "~" H 8700 3150 50  0001 C CNN
 	1    8700 3150
@@
 F 0 "D13" V 7746 3070 50  0000 R CNN
 F 1 "D" V 7655 3070 50  0000 R CNN
-F 2 "phase_v1_0:D_SOD-123-dual" H 7700 3150 50  0001 C CNN
+F 2 "phase:D_SOD-123-dual" H 7700 3150 50  0001 C CNN
 F 3 "~" H 7700 3150 50  0001 C CNN
 	1    7700 3150
@@
 F 0 "D14" V 8746 1570 50  0000 R CNN
 F 1 "D" V 8655 1570 50  0000 R CNN
-F 2 "phase_v1_0:D_SOD-123-dual" H 8700 1650 50  0001 C CNN
+F 2 "phase:D_SOD-123-dual" H 8700 1650 50  0001 C CNN
 F 3 "~" H 8700 1650 50  0001 C CNN
 	1    8700 1650
@@
 F 0 "D10" V 7746 1570 50  0000 R CNN
 F 1 "D" V 7655 1570 50  0000 R CNN
-F 2 "phase_v1_0:D_SOD-123-dual" H 7700 1650 50  0001 C CNN
+F 2 "phase:D_SOD-123-dual" H 7700 1650 50  0001 C CNN
 F 3 "~" H 7700 1650 50  0001 C CNN
 	1    7700 1650
@@
 F 0 "D7" V 6746 1570 50  0000 R CNN
 F 1 "D" V 6655 1570 50  0000 R CNN
-F 2 "phase_v1_0:D_SOD-123-dual" H 6700 1650 50  0001 C CNN
+F 2 "phase:D_SOD-123-dual" H 6700 1650 50  0001 C CNN
 F 3 "~" H 6700 1650 50  0001 C CNN
 	1    6700 1650
@@
 F 0 "D15" V 8746 2070 50  0000 R CNN
 F 1 "D" V 8655 2070 50  0000 R CNN
-F 2 "phase_v1_0:D_SOD-123-dual" H 8700 2150 50  0001 C CNN
+F 2 "phase:D_SOD-123-dual" H 8700 2150 50  0001 C CNN
 F 3 "~" H 8700 2150 50  0001 C CNN
 	1    8700 2150
@@
 F 0 "D11" V 7746 2070 50  0000 R CNN
 F 1 "D" V 7655 2070 50  0000 R CNN
-F 2 "phase_v1_0:D_SOD-123-dual" H 7700 2150 50  0001 C CNN
+F 2 "phase:D_SOD-123-dual" H 7700 2150 50  0001 C CNN
 F 3 "~" H 7700 2150 50  0001 C CNN
 	1    7700 2150
@@
 F 0 "D8" V 6746 2070 50  0000 R CNN
 F 1 "D" V 6655 2070 50  0000 R CNN
-F 2 "phase_v1_0:D_SOD-123-dual" H 6700 2150 50  0001 C CNN
+F 2 "phase:D_SOD-123-dual" H 6700 2150 50  0001 C CNN
 F 3 "~" H 6700 2150 50  0001 C CNN
 	1    6700 2150
@@
 F 0 "D16" V 8746 2570 50  0000 R CNN
 F 1 "D" V 8655 2570 50  0000 R CNN
-F 2 "phase_v1_0:D_SOD-123-dual" H 8700 2650 50  0001 C CNN
+F 2 "phase:D_SOD-123-dual" H 8700 2650 50  0001 C CNN
 F 3 "~" H 8700 2650 50  0001 C CNN
 	1    8700 2650
@@
 F 0 "D12" V 7746 2570 50  0000 R CNN
 F 1 "D" V 7655 2570 50  0000 R CNN
-F 2 "phase_v1_0:D_SOD-123-dual" H 7700 2650 50  0001 C CNN
+F 2 "phase:D_SOD-123-dual" H 7700 2650 50  0001 C CNN
 F 3 "~" H 7700 2650 50  0001 C CNN
 	1    7700 2650
@@
 F 0 "D9" V 6746 2570 50  0000 R CNN
 F 1 "D" V 6655 2570 50  0000 R CNN
-F 2 "phase_v1_0:D_SOD-123-dual" H 6700 2650 50  0001 C CNN
+F 2 "phase:D_SOD-123-dual" H 6700 2650 50  0001 C CNN
 F 3 "~" H 6700 2650 50  0001 C CNN
 	1    6700 2650
@@
 F 0 "D4" V 5746 1570 50  0000 R CNN
 F 1 "D" V 5655 1570 50  0000 R CNN
-F 2 "phase_v1_0:D_SOD-123-dual" H 5700 1650 50  0001 C CNN
+F 2 "phase:D_SOD-123-dual" H 5700 1650 50  0001 C CNN
 F 3 "~" H 5700 1650 50  0001 C CNN
 	1    5700 1650
@@
 F 0 "D5" V 5746 2070 50  0000 R CNN
 F 1 "D" V 5655 2070 50  0000 R CNN
-F 2 "phase_v1_0:D_SOD-123-dual" H 5700 2150 50  0001 C CNN
+F 2 "phase:D_SOD-123-dual" H 5700 2150 50  0001 C CNN
 F 3 "~" H 5700 2150 50  0001 C CNN
 	1    5700 2150
@@
 F 0 "D6" V 5746 2570 50  0000 R CNN
 F 1 "D" V 5655 2570 50  0000 R CNN
-F 2 "phase_v1_0:D_SOD-123-dual" H 5700 2650 50  0001 C CNN
+F 2 "phase:D_SOD-123-dual" H 5700 2650 50  0001 C CNN
 F 3 "~" H 5700 2650 50  0001 C CNN
 	1    5700 2650
@@
 F 0 "J2" H 5770 5083 50  0000 R CNN
 F 1 "AudioJack4" H 5770 5174 50  0000 R CNN
-F 2 "phase_v1_0:TRRS-PJ-320A-dual" H 6100 5200 50  0001 C CNN
+F 2 "phase:TRRS-PJ-320A-dual" H 6100 5200 50  0001 C CNN
 F 3 "~" H 6100 5200 50  0001 C CNN
 	1    6100 5200

Commit message: fix sda/scl swap, remove silkscreen art and unneeded ref des
Parts:
- J1: symbol Connector:USB_C_Receptacle_USB2.0 -> phase-rescue:USB_C_Receptacle_USB2.0-Connector
Connections:
- wire segments 163 -> 164
- no-connect marks 22 -> 25
Changed lines of the file:
@@
 encoding utf-8
 Sheet 1 1
-Title ""
+Title "Phase"
 Date ""
-Rev ""
+Rev "v1.0.1"
 Comp ""
 Comment1 ""
@@
 $EndComp
 $Comp
-L Connector:USB_C_Receptacle_USB2.0 J1
+L phase-rescue:USB_C_Receptacle_USB2.0-Connector J1
 U 1 1 5F4C922C
 P 1100 4900
@@
 	-1   0    0    1
 $EndComp
-Wire Wire Line
-	4600 5100 5100 5100
-Wire Wire Line
-	4600 5200 5300 5200
 $Comp
 L power:+5V #PWR015
@@
 Wire Wire Line
 	5100 5000 5100 5100
-Connection ~ 5100 5100
-Wire Wire Line
-	5100 5100 5900 5100
 Wire Wire Line
 	5300 5000 5300 5200
-Connection ~ 5300 5200
-Wire Wire Line
-	5300 5200 5900 5200
-Text Label 4700 5100 0    50   ~ 0
-SDA
-Text Label 4700 5200 0    50   ~ 0
+Text Label 5700 5200 0    50   ~ 0
 SCL
 $Comp
@@
 Wire Wire Line
 	8900 4800 9000 4800
-NoConn ~ 8900 4500
+NoConn ~ 9000 4500
 NoConn ~ 9000 4400
 Wire Wire Line
@@
 NoConn ~ 9000 5200
 NoConn ~ 9000 5300
-NoConn ~ 3200 2450
 NoConn ~ 8650 3600
 NoConn ~ 4700 4950
 Wire Wire Line
 	4600 6400 4700 6400
+Text Label 5700 5100 0    50   ~ 0
+SDA
+Text Label 4800 5200 2    50   ~ 0
+SDA
+Text Label 4800 5100 2    50   ~ 0
+SCL
+NoConn ~ 4700 6500
+NoConn ~ 4700 6600
+NoConn ~ 4700 6700
+NoConn ~ 4700 6800
+Wire Wire Line
+	9000 4500 8900 4500
+Wire Wire Line
+	5100 5100 5900 5100
+Wire Wire Line
+	5300 5200 5900 5200
+Wire Wire Line
+	4600 5100 4800 5100
+Wire Wire Line
+	4600 5200 4800 5200
 $EndSCHEMATC
